Commit message: add move to joint pose

File: models/franka_emika_panda/panda_arm.urdf (robot description, URDF)
Before this commit: robot panda, 9 links, 8 joints
Links:
- added link robotiq_payload, mass 1.05
Joints:
- added joint panda_robotiq_payload_joint: type fixed, parent panda_link8, child robotiq_payload, origin xyz=0 0 0 rpy=0 0 0

Commit message: add gravity ignore & change back to official urdf

File: models/franka_emika_panda/panda_arm.urdf (robot description, URDF)
Before this commit: robot panda, 10 links, 9 joints
Links:
- removed link robotiq_payload
Joints:
- removed joint panda_robotiq_payload_joint
